File: Electronics/Hardware/Standalone Board/displays.sch (KiCad schematic (older format))
At the start: 22 parts

Commit message: Everything is routed, TODO : lenghtmatching + impedance matching + cleaning
Parts:
- C61, C62, C63, C64, C65, C66, C67, C68, C69, C70, C71, C72: renamed from C?; footprint (none) -> Capacitor_SMD:C_0402_1005Metric
- J11, J12: renamed from J?; footprint (none) -> sb:FH35C-39S-0.3SHW(50)
- L4, L5, L7, L8: renamed from L?; footprint (none) -> sb:NRS8040T4R7NJGJ
- L6, L9: renamed from L?; footprint (none) -> sb:SDR0703
- U10, U9: renamed from U?; footprint (none) -> Package_DFN_QFN:WQFN-16-1EP_3x3mm_P0.5mm_EP1.75x1.75mm
